File: PCB/Teacup/Teacup.kicad_sch (KiCad schematic)
At the start: 90 parts, among them IC1 T31ZX, J1 USB Type-C, J2 SD_Card, J3 SFW15R-2STE1LF, J4 EXP0, J5 UART, J6 EXP2, J7 EXP1, J8 DC_IN, U1 AZ1117-3.3, U2 AZ1117-1.8, U3 MCP1826S, U4 W25Q32JVSS, U5 W25Q32JVSS, Y1 24 MHz

Commit message: pcb: boms and gerbers
Parts:
- C1, C10, C13, C16, C4, C7: footprint Capacitor_SMD:C_0603_1608Metric_Pad1.08x0.95mm_HandSolder -> Capacitor_SMD:C_0805_2012Metric_Pad1.18x1.45mm_HandSolder
- C20, C21: value TBD -> 12pF
- D1: Manufacturer (none) -> NXP; Manufacturer Part Number (none) -> PESD5V0U2BT,215
- IC1: Manufacturer (none) -> Lumissil; Manufacturer Part Number (none) -> T31ZX
- J1: Manufacturer Korean Hroparts Elec -> Korean Hroparts Elec (GTC); Manufacturer Part Number TYPE-C-31-M-12 -> TYPE-C-31-M-12 (USB4105-GF-A)
- J2: Manufacturer (none) -> Hirose; Manufacturer Part Number (none) -> DM1AA_SF_PEJ(82)
- J3: Manufacturer (none) -> Amphenol ICC; Manufacturer Part Number (none) -> SFW15R-2STE1LF
- J8: footprint (none) -> Connector_BarrelJack:BarrelJack_Wuerth_6941xx301002
- TP1, TP2, TP3, TP4, TP5, TP6, TP7, TP8, TP9: now left out of the parts list
- U1: Manufacturer (none) -> Diodes Incorporated; Manufacturer Part Number (none) -> AZ1117IH-3.3TRG1
- U2: Manufacturer (none) -> Diodes Incorporated; Manufacturer Part Number (none) -> AZ1117(CH)-1.8
- U3: Manufacturer (none) -> Microchip; Manufacturer Part Number (none) -> MCP1826S
- U4: Manufacturer (none) -> Winbond; Manufacturer Part Number (none) -> W25Q32JVSS
- Y1: Manufacturer (none) -> NDK; Manufacturer Part Number (none) -> NX2016SA-24MHZ-EXS00A-CS07553
